File: CAD/V1.0.0/Fuel_gauge_BQ27441.kicad_pcb (KiCad board)
At the start: 2 copper layers, 38 x 22 mm, 50 parts, among them K1 HEADER_MALE_1X1, K2 JST-2pin-SMD, K3 TERMINAL_KF235-5.0-2P, K4 easyC-SMD, K5 easyC-SMD, K6 HEADER_MALE_4X1, U1 BQ27441, U2 NMOS-DUAL, U3 SE5218

Commit message: Updating open source files.
Routing:
- net SCL3,3: track 38.6 -> 37.5 mm
Changed lines of the file:
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@@
   (gr_line (start 111 114) (end 147 114) (layer "Edge.Cuts") (width 0.1))
   (gr_line (start 110 93) (end 110 113) (layer "Edge.Cuts") (width 0.1))
-  (segment (start 126.438285 103.19) (end 125.41 103.19) (width 0.2) (layer "F.Cu") (net 1))
-  (segment (start 125.41 103.19) (end 125 103.6) (width 0.2) (layer "F.Cu") (net 1))
+  (segment (start 125.61 103.19) (end 126.438285 103.19) (width 0.2) (layer "F.Cu") (net 1))
+  (segment (start 125.3 103.5) (end 125.61 103.19) (width 0.2) (layer "F.Cu") (net 1))
   (via (at 115.2 105.2) (size 0.5) (drill 0.3) (layers "F.Cu" "B.Cu") (free) (net 1))
   (via (at 125.9 97.4) (size 0.5) (drill 0.3) (layers "F.Cu" "B.Cu") (free) (net 1))
   (via (at 124.1 98) (size 0.5) (drill 0.3) (layers "F.Cu" "B.Cu") (free) (net 1))
-  (via (at 125 103.6) (size 0.5) (drill 0.3) (layers "F.Cu" "B.Cu") (free) (net 1))
+  (via (at 125.3 103.5) (size 0.5) (drill 0.3) (layers "F.Cu" "B.Cu") (free) (net 1))
   (via (at 123.793541 101.884929) (size 0.5) (drill 0.3) (layers "F.Cu" "B.Cu") (free) (net 1))
   (segment (start 126.438285 103.99) (end 125.71 103.99) (width 0.2) (layer "F.Cu") (net 2))
@@
   (segment (start 124.65 99.15) (end 125.250489 98.549511) (width 0.4) (layer "F.Cu") (net 4))
   (segment (start 125.250489 97.550489) (end 124.95 97.25) (width 0.4) (layer "F.Cu") (net 4))
-  (segment (start 114.575978 101.1) (end 113.4 102.275978) (width 0.4) (layer "F.Cu") (net 5))
   (segment (start 119.60048 94.59952) (end 125 94.59952) (width 0.4) (layer "F.Cu") (net 5))
-  (segment (start 115.45 101.1) (end 114.575978 101.1) (width 0.4) (layer "F.Cu") (net 5))
   (segment (start 117.615 99.915) (end 117.615 98.715) (width 0.4) (layer "F.Cu") (net 5))
   (segment (start 120.2 99.15) (end 120.05 99) (width 0.4) (layer "F.Cu") (net 5))
   (segment (start 116.43 101.1) (end 115.45 101.1) (width 0.4) (layer "F.Cu") (net 5))
   (segment (start 117.615 98.715) (end 116.9 98) (width 0.4) (layer "F.Cu") (net 5))
-  (segment (start 113.4 106.8) (end 114.8 108.2) (width 0.4) (layer "F.Cu") (net 5))
+  (segment (start 113.2 106.824022) (end 114.575978 108.2) (width 0.4) (layer "F.Cu") (net 5))
   (segment (start 120.2 99.15) (end 118.72 99.15) (width 0.4) (layer "F.Cu") (net 5))
   (segment (start 126.4 100.25) (end 126.4 98.350978) (width 0.4) (layer "F.Cu") (net 5))
+  (segment (start 113.2 102.475978) (end 113.2 106.824022) (width 0.4) (layer "F.Cu") (net 5))
   (segment (start 120.4 108.2) (end 115.45 108.2) (width 0.4) (layer "F.Cu") (net 5))
+  (segment (start 115.45 101.1) (end 114.575978 101.1) (width 0.4) (layer "F.Cu") (net 5))
   (segment (start 129.22 98) (end 127.38 98) (width 0.4) (layer "F.Cu") (net 5))
   (segment (start 126.625489 98.125489) (end 126.750978 98) (width 0.4) (layer "F.Cu") (net 5))
@@
   (segment (start 116.9 98) (end 116.9 97.3) (width 0.4) (layer "F.Cu") (net 5))
   (segment (start 126.625489 96.225009) (end 126.625489 98.125489) (width 0.4) (layer "F.Cu") (net 5))
-  (segment (start 113.4 102.275978) (end 113.4 106.8) (width 0.4) (layer "F.Cu") (net 5))
   (segment (start 126.4 98.350978) (end 126.625489 98.125489) (width 0.4) (layer "F.Cu") (net 5))
+  (segment (start 114.575978 101.1) (end 113.2 102.475978) (width 0.4) (layer "F.Cu") (net 5))
   (segment (start 117.615 99.915) (end 116.43 101.1) (width 0.4) (layer "F.Cu") (net 5))
-  (segment (start 114.8 108.2) (end 115.45 108.2) (width 0.4) (layer "F.Cu") (net 5))
+  (segment (start 114.575978 108.2) (end 115.45 108.2) (width 0.4) (layer "F.Cu") (net 5))
   (segment (start 126.750978 98) (end 127.38 98) (width 0.4) (layer "F.Cu") (net 5))
   (segment (start 118.72 99.15) (end 118.6 99.03) (width 0.4) (layer "F.Cu") (net 5))
@@
   (segment (start 133.4 105.525) (end 133.125 105.525) (width 0.2) (layer "F.Cu") (net 12))
   (segment (start 130.388765 104.38952) (end 130.388285 104.39) (width 0.2) (layer "F.Cu") (net 12))
-  (segment (start 117.9 105.5) (end 117.181452 105.5) (width 0.4) (layer "F.Cu") (net 13))
-  (segment (start 115.45 103.768548) (end 115.45 103.1) (width 0.4) (layer "F.Cu") (net 13))
   (segment (start 119.225 109.925) (end 119.225 110.2) (width 0.4) (layer "F.Cu") (net 13))
-  (segment (start 117.181452 105.5) (end 115.45 103.768548) (width 0.4) (layer "F.Cu") (net 13))
   (segment (start 118.6 109.3) (end 119.225 109.925) (width 0.4) (layer "F.Cu") (net 13))
   (segment (start 127.38 95.28) (end 126.1 94) (width 0.4) (layer "F.Cu") (net 13))
+  (segment (start 117.369037 105.149511) (end 116.449511 105.149511) (width 0.4) (layer "F.Cu") (net 13))
+  (segment (start 116.449511 105.149511) (end 115.4 104.1) (width 0.4) (layer "F.Cu") (net 13))
+  (segment (start 115.4 103.15) (end 115.45 103.1) (width 0.4) (layer "F.Cu") (net 13))
+  (segment (start 117.434274 105.084274) (end 117.369037 105.149511) (width 0.4) (layer "F.Cu") (net 13))
   (segment (start 115.5 103.15) (end 115.45 103.1) (width 0.4) (layer "F.Cu") (net 13))
   (segment (start 118.6 109.3) (end 117.7 110.2) (width 0.4) (layer "F.Cu") (net 13))
   (segment (start 126.1 94) (end 119.2 94) (width 0.4) (layer "F.Cu") (net 13))
   (segment (start 119.2 94) (end 112.7 100.5) (width 0.4) (layer "F.Cu") (net 13))
-  (segment (start 114.0495 104.1) (end 114.45 104.1) (width 0.4) (layer "F.Cu") (net 13))
   (segment (start 117.7 110.2) (end 115.45 110.2) (width 0.4) (layer "F.Cu") (net 13))
+  (segment (start 114.0495 103.1) (end 115.45 103.1) (width 0.4) (layer "F.Cu") (net 13))
+  (segment (start 117.85 105.5) (end 117.434274 105.084274) (width 0.4) (layer "F.Cu") (net 13))
   (segment (start 127.38 97.35) (end 127.38 95.28) (width 0.4) (layer "F.Cu") (net 13))
-  (segment (start 114.45 104.1) (end 115.45 103.1) (width 0.4) (layer "F.Cu") (net 13))
+  (segment (start 117.9 105.5) (end 117.85 105.5) (width 0.4) (layer "F.Cu") (net 13))
+  (segment (start 115.4 104.1) (end 115.4 103.15) (width 0.4) (layer "F.Cu") (net 13))
   (via (at 117.9 105.5) (size 0.5) (drill 0.3) (layers "F.Cu" "B.Cu") (net 13))
   (via (at 112.7 100.5) (size 0.5) (drill 0.3) (layers "F.Cu" "B.Cu") (net 13))
   (via (at 118.6 109.3) (size 0.5) (drill 0.3) (layers "F.Cu" "B.Cu") (net 13))
-  (via (at 114.0495 104.1) (size 0.5) (drill 0.3) (layers "F.Cu" "B.Cu") (net 13))
+  (via (at 114.0495 103.1) (size 0.5) (drill 0.3) (layers "F.Cu" "B.Cu") (net 13))
   (segment (start 118.6 109.3) (end 117.9 108.6) (width 0.4) (layer "B.Cu") (net 13))
   (segment (start 117.9 108.6) (end 117.9 105.5) (width 0.4) (layer "B.Cu") (net 13))
-  (segment (start 112.7 100.5) (end 112.7 102.7505) (width 0.4) (layer "B.Cu") (net 13))
-  (segment (start 112.7 102.7505) (end 114.0495 104.1) (width 0.4) (layer "B.Cu") (net 13))
+  (segment (start 114.0495 103.1) (end 112.7 101.7505) (width 0.4) (layer "B.Cu") (net 13))
+  (segment (start 112.7 101.7505) (end 112.7 100.5) (width 0.4) (layer "B.Cu") (net 13))
   (segment (start 129.22 99.78) (end 129.22 98.65) (width 0.2) (layer "F.Cu") (net 14))
   (segment (start 128.9 100.1) (end 129.22 99.78) (width 0.2) (layer "F.Cu") (net 14))
@@
   (zone (net 12) (net_name "VSYS") (layer "F.Cu") (hatch edge 0.508)
     (priority 3)
-    (connect_pads (clearance 0.254))
+    (connect_pads yes (clearance 0.254))
     (min_thickness 0.254) (filled_areas_thickness no)
     (fill yes (thermal_gap 0.508) (thermal_bridge_width 0.508))
     (polygon
       (pts
-        (xy 144.8 107.4)
-        (xy 137.2 107.4)
-        (xy 134.8 109.8)
-        (xy 133.6 109.8)
-        (xy 133.6 106.4)
-        (xy 131.8 106.4)
-        (xy 131.8 104.4)
-        (xy 144.8 104.4)
+        (xy 144.7 106.9)
+        (xy 144 107.6)
+        (xy 136.2 107.6)
+        (xy 134.5 109.3)
+        (xy 133.8 109.3)
+        (xy 133.8 106.8)
+        (xy 133.1 106.1)
+        (xy 132.5 106.1)
+        (xy 132.5 105)
+        (xy 134.3 105)
+        (xy 135.3 104.7)
+        (xy 144 104.7)
+        (xy 144.7 105.4)
       )
     )
@@
   (zone (net 3) (net_name "VCC") (layer "F.Cu") (hatch edge 0.508)
     (priority 3)
-    (connect_pads (clearance 0.254))
+    (connect_pads yes (clearance 0.254))
     (min_thickness 0.254) (filled_areas_thickness no)
     (fill yes (thermal_gap 0.508) (thermal_bridge_width 0.508))
     (polygon
       (pts
-        (xy 139.2 102)
-        (xy 138.996721 102.963935)
-        (xy 132.696299 103.744377)
-        (xy 131.481573 101.983763)
-        (xy 131.266789 100.085061)
-        (xy 134.9 100.09)
-        (xy 135.4 102)
-        (xy 137.6 102)
-        (xy 137.6 99.4)
-        (xy 139.2 99.4)
+        (xy 139 102)
+        (xy 138 102.963935)
+        (xy 132.5 103)
+        (xy 131.7 102.2)
+        (xy 131.7 100.5)
+        (xy 132.7 100.5)
+        (xy 134.1 101.9)
+        (xy 137.4 101.9)
+        (xy 137.8 101.5)
+        (xy 137.8 99.6)
+        (xy 139 99.6)
       )
     )
